File: kicad/slckb/slckb.sch (KiCad schematic (older format))
At the start: 15 parts, among them J1 Conn_01x04, J2 Conn_01x08, J3 Conn_01x16, U1 ATmega32U4-AU, U2 74AHC138, U3 74AHC138, Y1 Crystal_GND24

Commit message: removed bak files, updated TODO
Parts:
- added C5: 4u7, symbol Device:C
Connections:
- net GNDD: now also C5.2
- net VBUS: now also C5.1
Changed lines of the file:
@@
 	1    0    0    -1
 $EndComp
+$Comp
+L Device:C C5
+U 1 1 5FA20CA3
+P 2100 1250
+F 0 "C5" H 2215 1296 50  0000 L CNN
+F 1 "4u7" H 2215 1205 50  0000 L CNN
+F 2 "" H 2138 1100 50  0001 C CNN
+F 3 "~" H 2100 1250 50  0001 C CNN
+	1    2100 1250
+	1    0    0    -1
+$EndComp
+Connection ~ 2100 1100
+Connection ~ 2100 1400
 $EndSCHEMATC

Commit message: general update
Parts:
- added C?: 100n, symbol Device:C
- R1, R2: footprint 22R -> (none)
Connections:
- net GNDD: now also C?.1
- net VBUS: now also C?.2
Other:
- note added: "Dodaj globalny Enable\ntylko czy potrzebny?\n"
Changed lines of the file:
@@
 F 0 "R1" V 693 4700 50  0000 C CNN
 F 1 "22R" V 784 4700 50  0000 C CNN
-F 2 "22R" V 830 4700 50  0001 C CNN
+F 2 "" V 830 4700 50  0001 C CNN
 F 3 "~" H 900 4700 50  0001 C CNN
 	1    900  4700
@@
 F 0 "R2" V 1100 4800 50  0000 C CNN
 F 1 "22R" V 1000 4800 50  0000 C CNN
-F 2 "22R" V 830 4800 50  0001 C CNN
+F 2 "" V 830 4800 50  0001 C CNN
 F 3 "~" H 900 4800 50  0001 C CNN
 	1    900  4800
@@
 Wire Wire Line
 	3550 6000 3550 4350
-Wire Wire Line
-	3950 6200 3950 6100
 $Comp
 L power:VBUS #PWR012
@@
 $EndComp
 $Comp
-L power:GNDD #PWR010
-U 1 1 5FAA5855
-P 3950 4450
-F 0 "#PWR010" H 3950 4200 50  0001 C CNN
-F 1 "GNDD" H 3954 4295 50  0000 C CNN
-F 2 "" H 3950 4450 50  0001 C CNN
-F 3 "" H 3950 4450 50  0001 C CNN
-	1    3950 4450
-	1    0    0    -1
-$EndComp
-$Comp
 L power:GNDD #PWR013
 U 1 1 5FAA678E
@@
 	1    0    0    -1
 $EndComp
-Connection ~ 3950 6200
 Wire Wire Line
 	3250 3850 3750 3850
@@
 Connection ~ 2100 1100
 Connection ~ 2100 1400
+Text Notes 3050 6300 0    50   ~ 0
+Dodaj globalny Enable\ntylko czy potrzebny?\n
+Wire Wire Line
+	3950 6200 3950 6100
+Connection ~ 3950 6200
+$Comp
+L power:GNDD #PWR0101
+U 1 1 5FA39CD3
+P 3950 4450
+F 0 "#PWR0101" H 3950 4200 50  0001 C CNN
+F 1 "GNDD" H 3954 4295 50  0000 C CNN
+F 2 "" H 3950 4450 50  0001 C CNN
+F 3 "" H 3950 4450 50  0001 C CNN
+	1    3950 4450
+	1    0    0    -1
+$EndComp
+$Comp
+L Device:C C?
+U 1 1 5FA42907
+P 2100 3400
+F 0 "C?" V 1848 3400 50  0000 C CNN
+F 1 "100n" V 1939 3400 50  0000 C CNN
+F 2 "" H 2138 3250 50  0001 C CNN
+F 3 "~" H 2100 3400 50  0001 C CNN
+	1    2100 3400
+	0    1    1    0
+$EndComp
+Connection ~ 1950 3400
+$Comp
+L power:GNDD #PWR?
+U 1 1 5FA43FFD
+P 2250 3400
+F 0 "#PWR?" H 2250 3150 50  0001 C CNN
+F 1 "GNDD" H 2254 3245 50  0000 C CNN
+F 2 "" H 2250 3400 50  0001 C CNN
+F 3 "" H 2250 3400 50  0001 C CNN
+	1    2250 3400
+	0    -1   -1   0
+$EndComp
 $EndSCHEMATC

Commit message: some updates
Parts:
- J2: value Conn_01x08 -> 01x08
- gave numbers to parts that had none: 1
