File: kicad/sw_pcb/sw_pcb.sch (KiCad schematic (older format))
At the start: 144 parts, among them J1 Conn_01x08, J2 Conn_01x09, SW1 SW, SW10 SW, SW11 SW, SW12 SW, SW13 SW, SW14 SW, SW15 SW, SW16 SW, SW17 SW, SW18 SW, SW19 SW, SW2 SW, SW20 SW, SW21 SW, SW22 SW, SW23 SW, SW24 SW, SW25 SW, SW26 SW, SW27 SW, SW28 SW, SW29 SW, SW3 SW, SW30 SW, SW31 SW, SW32 SW, SW33 SW, SW34 SW, SW35 SW, SW36 SW, SW37 SW, SW38 SW, SW39 SW, SW4 SW, SW40 SW, SW41 SW, SW42 SW, SW43 SW, SW44 SW, SW45 SW, SW46 SW, SW47 SW, SW48 SW, SW49 SW, SW5 SW, SW50 SW, SW51 SW, SW52 SW, SW53 SW, SW54 SW, SW55 SW, SW56 SW, SW57 SW, SW58 SW, SW59 SW, SW6 SW, SW60 SW, SW61 SW, SW62 SW, SW63 SW, SW64 SW, SW65 SW, SW66 SW, SW67 SW, SW68 SW, SW69 SW, SW7 SW, SW70 SW, SW71 SW, SW8 SW, SW9 SW

Commit message: some updates
Parts:
- D1, D10, D11, D12, D13, D14, D15, D16, D17, D18, D19, D2, D20, D21, D22, D23, D24, D25, D26, D27, D28, D29, D3, D30, D31, D32, D33, D34, D35, D36, D37, D38, D39, D4, D40, D41, D42, D43, D44, D45, D46, D47, D48, D49, D5, D50, D51, D52, D53, D54, D55, D56, D57, D58, D59, D6, D60, D61, D62, D63, D64, D65, D66, D67, D68, D69, D7, D70, D71, D8, D9: footprint (none) -> Diode_SMD:D_MicroMELF
- J1: footprint (none) -> Connector_PinSocket_2.54mm:PinSocket_1x08_P2.54mm_Vertical
- SW1, SW10, SW11, SW12, SW13, SW14, SW15, SW16, SW17, SW18, SW19, SW2, SW20, SW21, SW22, SW23, SW24, SW25, SW26, SW27, SW28, SW29, SW3, SW30, SW31, SW32, SW33, SW34, SW35, SW36, SW37, SW38, SW39, SW4, SW40, SW41, SW42, SW43, SW44, SW45, SW46, SW47, SW48, SW49, SW5, SW50, SW51, SW52, SW53, SW54, SW55, SW56, SW57, SW58, SW59, SW6, SW60, SW61, SW62, SW63, SW64, SW65, SW66, SW67, SW68, SW69, SW7, SW70, SW71, SW8, SW9: footprint (none) -> Button_Switch_Keyboard:SW_Cherry_MX_1.00u_PCB
